File: pico_tracker_v3.1.brd (EAGLE design)
At the start: 58.4 x 34.3 mm, 28 parts, among them Q1 CSTCR6M00G53Z, Q2 4 MHz, U1 ATMEGA328, U2 MCP1640

Commit message: New version of PCB and power safe mode for GPS
Parts:
- R6: value 820k -> 430k
- R8: value 430k -> 820k
Changed lines of the file:
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@@
 <attribute name="VALUE" x="56.7055" y="43.6118" size="1.27" layer="21" font="vector" rot="R270"/>
 </element>
-<element name="R6" library="resistor" package="R0603" value="820k" x="52.3875" y="44.1325" smashed="yes" rot="MR180">
+<element name="R6" library="resistor" package="R0603" value="430k" x="52.3875" y="44.1325" smashed="yes" rot="MR180">
 <attribute name="NAME" x="54.4449" y="44.6405" size="0.762" layer="26" font="vector" rot="MR180"/>
 </element>
-<element name="R8" library="resistor" package="R0603" value="430k" x="49.8475" y="44.1325" smashed="yes" rot="MR180">
+<element name="R8" library="resistor" package="R0603" value="820k" x="49.8475" y="44.1325" smashed="yes" rot="MR180">
 <attribute name="NAME" x="46.1391" y="44.4119" size="0.762" layer="26" font="vector" rot="MR180"/>
 </element>
