File: pico_tracker_v3.1.sch (EAGLE design)
At the start: 28 parts, among them Q1 CSTCR6M00G53Z, Q2 4 MHz, U1 ATMEGA328, U2 MCP1640, X1 87758-1416

Commit message: New version of PCB and power safe mode for GPS
Parts:
- R6: value 820k -> 430k
- R8: value 430k -> 820k
Changed lines of the file:
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@@
 <part name="GND12" library="SparkFun" deviceset="GND" device=""/>
 <part name="JP1" library="SparkFun" deviceset="M02" device="PTH" value="Battery"/>
-<part name="R6" library="resistor" deviceset="R-EU_" device="R0603" value="820k"/>
-<part name="R8" library="resistor" deviceset="R-EU_" device="R0603" value="430k"/>
+<part name="R6" library="resistor" deviceset="R-EU_" device="R0603" value="430k"/>
+<part name="R8" library="resistor" deviceset="R-EU_" device="R0603" value="820k"/>
 <part name="Q2" library="ava" deviceset="ABRACON_ABM3_CRYSTAL" device="ABM03_HC49" value="4 MHz"/>
 <part name="C4" library="resistor" deviceset="C-EU" device="C0603" value="16p"/>
